File: hardware/pcb/flight_computer/mcu.kicad_sch (KiCad schematic)
At the start: 1 part, among them U6 Teensy4.1

Commit message: Added 3D model
Connections:
- no-connect marks 0 -> 25
Changed lines of the file:
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@@
 		(color 0 0 0 0)
+	)
+	(no_connect
+		(at 116.84 128.27)
+	)
+	(no_connect
+		(at 172.72 133.35)
+	)
+	(no_connect
+		(at 172.72 66.04)
+	)
+	(no_connect
+		(at 172.72 52.07)
+	)
+	(no_connect
+		(at 172.72 120.65)
+	)
+	(no_connect
+		(at 116.84 96.52)
+	)
+	(no_connect
+		(at 137.16 143.51)
+	)
+	(no_connect
+		(at 116.84 119.38)
+	)
+	(no_connect
+		(at 116.84 121.92)
+	)
+	(no_connect
+		(at 172.72 63.5)
+	)
+	(no_connect
+		(at 172.72 128.27)
+	)
+	(no_connect
+		(at 116.84 125.73)
+	)
+	(no_connect
+		(at 116.84 130.81)
+	)
+	(no_connect
+		(at 116.84 68.58)
+	)
+	(no_connect
+		(at 116.84 101.6)
+	)
+	(no_connect
+		(at 116.84 93.98)
+	)
+	(no_connect
+		(at 172.72 125.73)
+	)
+	(no_connect
+		(at 116.84 99.06)
+	)
+	(no_connect
+		(at 116.84 91.44)
+	)
+	(no_connect
+		(at 172.72 60.96)
+	)
+	(no_connect
+		(at 116.84 71.12)
+	)
+	(no_connect
+		(at 172.72 130.81)
+	)
+	(no_connect
+		(at 152.4 143.51)
+	)
+	(no_connect
+		(at 140.97 143.51)
+	)
+	(no_connect
+		(at 148.59 143.51)
 	)
 	(wire
