File: hardware/pcb/flight_computer/mcu.kicad_sch (KiCad schematic)
At the start: 1 part, among them U6 Teensy4.1

Commit message: Consolidate simulation and hardware into single ember repo
Absorb the standalone simulation repo into ember as plain files,
add root .gitignore, and update hardware CAD assets.

Co-Authored-By: Claude Opus 4.8 <noreply@anthropic.com>
Connections:
- net CE_NRF: now also U6.22 (30_CRX3); no longer U6.23 (31_CTX3)
- net CNS_NRF: now also U6.23 (31_CTX3); no longer U6.22 (30_CRX3)
- net CONT_1: now also U6.33 (41_A17); no longer U6.32 (40_A16)
- net CONT_2: now also U6.32 (40_A16); no longer U6.33 (41_A17)
- net CS_IMU: now also U6.11 (9_OUT1C); no longer U6.10 (8_TX2_IN1)
- net FIRE_1: now also U6.25 (33_MCLK2); no longer U6.28 (36_CS)
- net FIRE_2: now also U6.28 (36_CS); no longer U6.29 (37_CS)
- net INT_IMU_2: now also U6.10 (8_TX2_IN1); no longer U6.11 (9_OUT1C)
- net LED_B: now also U6.29 (37_CS); no longer U6.25 (33_MCLK2)
- net GPIO_1: no longer names the net of U6.5 (3_LRCLK2)
- net GPIO_2: no longer names the net of U6.4 (2_OUT2)
