File: hardware/pcb/flight_computer/flight_computer.kicad_sch (KiCad schematic)
At the start: 12 parts, among them J2 BATT_TERMINAL, J3 5V Terminal, J4 Pyro 1, J5 Pyro 2, J8 Conn_01x02, J9 Aux Ports

Commit message: Consolidate simulation and hardware into single ember repo
Absorb the standalone simulation repo into ember as plain files,
add root .gitignore, and update hardware CAD assets.

Co-Authored-By: Claude Opus 4.8 <noreply@anthropic.com>
Parts:
- removed J8: Conn_01x02, Connector_PinHeader_2.54mm:PinHeader_1x02_P2.54mm_Vertical, symbol Connector_Generic:Conn_01x02
Connections:
- net Pyro 1/PYRO+: now also J4.1 (Pin_1); no longer J4.2 (Pin_2)
- net Pyro 1/PYRO-: now also J4.2 (Pin_2); no longer J4.1 (Pin_1)
- net Pyro 2/PYRO+: now also J5.1 (Pin_1); no longer J5.2 (Pin_2)
- net Pyro 2/PYRO-: now also J5.2 (Pin_2); no longer J5.1 (Pin_1)
- net SCL: now also J9.3 (Pin_3); no longer J9.5 (Pin_5)
- net SDA: now also J9.5 (Pin_5); no longer J9.3 (Pin_3)
Other:
- sheet MCU ports: added none; removed GPIO_1, GPIO_2
Changed lines of the file:
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@@
 	(wire
 		(pts
+			(xy 64.77 138.43) (xy 95.25 138.43)
+		)
+		(stroke
+			(width 0)
+			(type default)
+		)
+	)
+	(wire
+		(pts
 			(xy 72.39 187.96) (xy 97.79 187.96)
 		)
@@
 	(wire
 		(pts
+			(xy 64.77 168.91) (xy 95.25 168.91)
+		)
+		(stroke
+			(width 0)
+			(type default)
+		)
+	)
+	(wire
+		(pts
+			(xy 64.77 166.37) (xy 95.25 166.37)
+		)
+		(stroke
+			(width 0)
+			(type default)
+		)
+	)
+	(wire
+		(pts
 			(xy 105.41 43.18) (xy 105.41 45.72)
 		)
@@
 	(wire
 		(pts
-			(xy 64.77 168.91) (xy 95.25 168.91)
-		)
-		(stroke
-			(width 0)
-			(type default)
-		)
-	)
-	(wire
-		(pts
 			(xy 193.04 91.44) (xy 217.17 91.44)
 		)
@@
 	(wire
 		(pts
-			(xy 64.77 138.43) (xy 95.25 138.43)
+			(xy 200.66 151.13) (xy 213.36 151.13)
 		)
 		(stroke
@@
 	(wire
 		(pts
-			(xy 193.04 123.19) (xy 207.01 123.19)
+			(xy 200.66 148.59) (xy 213.36 148.59)
 		)
 		(stroke
@@
 	(wire
 		(pts
-			(xy 64.77 166.37) (xy 95.25 166.37)
-		)
-		(stroke
-			(width 0)
-			(type default)
-		)
-	)
-	(wire
-		(pts
 			(xy 233.68 156.21) (xy 233.68 153.67)
 		)
@@
 	(wire
 		(pts
-			(xy 171.45 147.32) (xy 181.61 147.32)
+			(xy 64.77 135.89) (xy 95.25 135.89)
 		)
 		(stroke
@@
 	(wire
 		(pts
-			(xy 171.45 149.86) (xy 181.61 149.86)
-		)
-		(stroke
-			(width 0)
-			(type default)
-		)
-	)
-	(wire
-		(pts
-			(xy 200.66 151.13) (xy 213.36 151.13)
-		)
-		(stroke
-			(width 0)
-			(type default)
-		)
-	)
-	(wire
-		(pts
 			(xy 115.57 92.71) (xy 152.4 92.71)
 		)
@@
 	(wire
 		(pts
-			(xy 64.77 135.89) (xy 95.25 135.89)
-		)
-		(stroke
-			(width 0)
-			(type default)
-		)
-	)
-	(wire
-		(pts
 			(xy 217.17 62.23) (xy 233.68 62.23)
 		)
@@
 	(wire
 		(pts
-			(xy 193.04 120.65) (xy 207.01 120.65)
-		)
-		(stroke
-			(width 0)
-			(type default)
-		)
-	)
-	(wire
-		(pts
-			(xy 200.66 148.59) (xy 213.36 148.59)
-		)
-		(stroke
-			(width 0)
-			(type default)
-		)
-	)
-	(wire
-		(pts
 			(xy 113.03 163.83) (xy 123.19 163.83)
 		)
@@
 		)
 	)
-	(label "GPIO_1"
-		(at 207.01 120.65 180)
-		(effects
-			(font
-				(size 1.27 1.27)
-			)
-			(justify right bottom)
-		)
-	)
 	(label "FIRE_1"
 		(at 134.62 114.3 0)
@@
 	)
 	(label "SCL"
-		(at 200.66 151.13 0)
+		(at 200.66 148.59 0)
 		(effects
 			(font
@@
 		)
 	)
-	(label "GPIO_1"
-		(at 181.61 147.32 180)
-		(effects
-			(font
-				(size 1.27 1.27)
-			)
-			(justify right bottom)
-		)
-	)
 	(label "TX_GPS"
 		(at 237.49 151.13 180)
@@
 		)
 	)
-	(label "GPIO_2"
-		(at 207.01 123.19 180)
-		(effects
-			(font
-				(size 1.27 1.27)
-			)
-			(justify right bottom)
-		)
-	)
 	(label "CS_BARO"
 		(at 207.01 78.74 180)
@@
 		)
 	)
-	(label "GPIO_2"
-		(at 181.61 149.86 180)
-		(effects
-			(font
-				(size 1.27 1.27)
-			)
-			(justify right bottom)
-		)
-	)
 	(label "CE_NRF"
 		(at 207.01 63.5 180)
@@
 	)
 	(label "SDA"
-		(at 200.66 148.59 0)
+		(at 200.66 151.13 0)
 		(effects
 			(font
@@
 	)
 	(symbol
-		(lib_id "Connector_Generic:Conn_01x02")
-		(at 166.37 149.86 180)
-		(unit 1)
-		(body_style 1)
-		(exclude_from_sim no)
-		(in_bom yes)
-		(on_board yes)
-		(in_pos_files yes)
-		(dnp no)
-		(fields_autoplaced yes)
-		(property "Reference" "J8"
-			(at 166.37 140.97 0)
-			(show_name no)
-			(do_not_autoplace no)
-			(effects
-				(font
-					(size 1.27 1.27)
-				)
-			)
-		)
-		(property "Value" "Conn_01x02"
-			(at 166.37 143.51 0)
-			(show_name no)
-			(do_not_autoplace no)
-			(effects
-				(font
-					(size 1.27 1.27)
-				)
-			)
-		)
-		(property "Footprint" "Connector_PinHeader_2.54mm:PinHeader_1x02_P2.54mm_Vertical"
-			(at 166.37 149.86 0)
-			(hide yes)
-			(show_name no)
-			(do_not_autoplace no)
-			(effects
-				(font
-					(size 1.27 1.27)
-				)
-			)
-		)
-		(property "Datasheet" ""
-			(at 166.37 149.86 0)
-			(hide yes)
-			(show_name no)
-			(do_not_autoplace no)
-			(effects
-				(font
-					(size 1.27 1.27)
-				)
-			)
-		)
-		(property "Description" "Generic connector, single row, 01x02, script generated (kicad-library-utils/schlib/autogen/connector/)"
-			(at 166.37 149.86 0)
-			(hide yes)
-			(show_name no)
-			(do_not_autoplace no)
-			(effects
-				(font
-					(size 1.27 1.27)
-				)
-			)
-		)
-		(pin "2"
-		)
-		(pin "1"
-		)
-		(instances
-			(project "flight_computer"
-				(path "/97739cb3-517e-4f70-8350-1cb198e6b8e6"
-					(reference "J8")
-					(unit 1)
-				)
-			)
-		)
-	)
-	(symbol
 		(lib_id "power:GND")
 		(at 36.83 81.28 0)
@@
 			)
 		)
-		(pin "GPIO_1" bidirectional
-			(at 193.04 120.65 0)
-			(effects
-				(font
-					(size 1.27 1.27)
-				)
-				(justify right)
-			)
-		)
-		(pin "GPIO_2" bidirectional
-			(at 193.04 123.19 0)
-			(effects
-				(font
-					(size 1.27 1.27)
-				)
-				(justify right)
-			)
-		)
 		(instances
 			(project "flight_computer"
@@
 		)
 		(pin "PYRO+" output
-			(at 95.25 135.89 180)
+			(at 95.25 138.43 180)
 			(effects
 				(font
@@
 		)
 		(pin "PYRO-" output
-			(at 95.25 138.43 180)
+			(at 95.25 135.89 180)
 			(effects
 				(font
@@
 		)
 		(pin "PYRO+" output
-			(at 95.25 166.37 180)
+			(at 95.25 168.91 180)
 			(effects
 				(font
@@
 		)
 		(pin "PYRO-" output
-			(at 95.25 168.91 180)
+			(at 95.25 166.37 180)
 			(effects
 				(font
