File: hardware/pcb/flight_computer/power.kicad_sch (KiCad schematic)
At the start: 30 parts, among them U2 TPS563201DDCR, U3 TPS73633DRBR, U7 AZ1117-5.0

Commit message: Consolidate simulation and hardware into single ember repo
Absorb the standalone simulation repo into ember as plain files,
add root .gitignore, and update hardware CAD assets.

Co-Authored-By: Claude Opus 4.8 <noreply@anthropic.com>
Parts:
- U3: footprint footprints:IC_DRV8601DRBT -> footprints:SOT95P280X145-5N
Connections:
- net +3.3V: now also U3.5 (OUT); no longer U3.1 (OUT)
- net +5V: now also U3.1 (IN), U3.3 (EN), U7.4 (VOUT); no longer U3.5 (EN), U3.8 (IN)
- net GND: now also U3.2 (GND); no longer U3.4 (GND)
- net at C9.1: now also U3.4 (NR/FB); no longer U3.3 (NR/FB)
Other:
- moved on the sheet: C21
